Commit message: Tekerlekler gün yüzüne çıktı

File: wheelchair_description/urdf/wheel_chair.urdf.xacro (robot description, xacro)
@@ -7,5 +7,5 @@
     <parent link="base_footprint" />
     <child link="base_link" />
-    <origin xyz="0.0 0.0 0.0010" rpy="0 0 0" />
+    <origin xyz="0.0 0.0 0.15345" rpy="0 0 0" />
   </joint>
   <link

Commit message: gereksizler silindi, fgm ye gore duzenlemeler yapildi

File: wheelchair_description/urdf/wheel_chair.urdf.xacro (robot description, xacro)
@@ -7,5 +7,5 @@
     <parent link="base_footprint" />
     <child link="base_link" />
-    <origin xyz="0.0 0.0 0.15345" rpy="0 0 0" />
+    <origin xyz="-0.40 0.0 0.15345" rpy="0 0 0" />
   </joint>
   <link

Commit message: gap merge işlemi yapıldı, hafızadaki ayrı gapler koordinatları ile birlikte mevcut

File: wheelchair_description/urdf/wheel_chair.urdf.xacro (robot description, xacro)
@@ -3,5 +3,11 @@
   <!-- <xacro:include filename="$(find turtlebot3_description)/urdf/common_properties.xacro" /> -->
   <xacro:include filename="$(find wheelchair_description)/urdf/wheel_chair.gazebo.xacro" />
-  <link name="base_footprint" />
+  <link name="base_footprint" >
+    <visual>
+      <geometry>
+        <cylinder length = "0.2" radius="0.05" />
+      </geometry>
+    </visual>
+</link>
   <joint name="base_joint" type="fixed">
     <parent link="base_footprint" />
