Commit message: Ön tekerlekler problemli

File: wheelchair_description/urdf/wheel_chair.gazebo.xacro (robot description, xacro)
@@ -26,5 +26,5 @@
     <material>Gazebo/FlatBlack</material>
   </gazebo>
-  <gazebo reference="left_small_wheel">
+<!--   <gazebo reference="left_small_wheel">
     <mu1>0.1</mu1>
     <mu2>0.1</mu2>
@@ -34,6 +34,6 @@
     <maxVel>1.0</maxVel>
     <material>Gazebo/FlatBlack</material>
-  </gazebo>
-  <gazebo reference="right_smaal_wheel">
+  </gazebo> -->
+ <!--  <gazebo reference="right_smaal_wheel">
     <mu1>0.1</mu1>
     <mu2>0.1</mu2>
@@ -43,5 +43,5 @@
     <maxVel>1.0</maxVel>
     <material>Gazebo/FlatBlack</material>
-  </gazebo>
+  </gazebo> -->
   <gazebo reference="imu_link">
     <sensor type="imu" name="imu">
@@ -52,5 +52,5 @@
   </gazebo>
   <gazebo>
-    <plugin name="turtlebot3_burger_controller" filename="libgazebo_ros_diff_drive.so">
+    <plugin name="wheel_chair_controller" filename="libgazebo_ros_diff_drive.so">
       <commandTopic>cmd_vel</commandTopic>
       <odometryTopic>odom</odometryTopic>
@@ -65,5 +65,7 @@
       <updateRate>30</updateRate>
       <leftJoint>left_big_wheel_joint</leftJoint>
+      <!-- <leftJoint>left_small_wheel_joint</leftJoint> -->
       <rightJoint>right_big_wheel_joint</rightJoint>
+      <!-- <rightJoint>right_small_wheel_joint</rightJoint> -->
       <wheelSeparation>0.575</wheelSeparation>
       <wheelDiameter>0.324</wheelDiameter>
@@ -102,6 +104,6 @@
   </gazebo>
   <gazebo reference="rp_laser_front">
-    <material>Gazebo/FlatBlack</material>
-    <sensor type="ray" name="lds_lfcd_sensor">
+    <material>Gazebo/RedBright</material>
+    <sensor type="ray" name="lds_lfcd_sensor_front">
       <pose>0.00386881875434386 8.69539989361567E-05 -0.00554963797433417 0 0 0</pose>
       <visualize>$(arg laser_visual)</visualize>
@@ -127,5 +129,5 @@
         </noise>
       </ray>
-      <plugin name="gazebo_ros_lds_lfcd_controller" filename="libgazebo_ros_laser.so">
+      <plugin name="gazebo_ros_lds_lfcd_controller_front" filename="libgazebo_ros_laser.so">
         <topicName>front_rp/rp_scan_filtered_front/</topicName>
         <frameName>rp_laser_front</frameName>
@@ -133,3 +135,35 @@
     </sensor>
   </gazebo>
+  <gazebo reference="rp_laser_back">
+    <material>Gazebo/Gold</material>
+    <sensor type="ray" name="lds_lfcd_sensor_back">
+      <pose>-0.00393393719392465 1.45541326387055E-05 -0.00550433759472346 0 0 0</pose>
+      <visualize>$(arg laser_visual)</visualize>
+      <update_rate>10</update_rate>
+      <ray>
+        <scan>
+          <horizontal>
+            <samples>360</samples>
+            <resolution>1</resolution>
+            <min_angle>0.0</min_angle>
+            <max_angle>6.28319</max_angle>
+          </horizontal>
+        </scan>
+        <range>
+          <min>0.12</min>
+          <max>7.0</max>
+          <resolution>0.015</resolution>
+        </range>
+        <noise>
+          <type>gaussian</type>
+          <mean>0.0</mean>
+          <stddev>0.01</stddev>
+        </noise>
+      </ray>
+      <plugin name="gazebo_ros_lds_lfcd_controller_back" filename="libgazebo_ros_laser.so">
+        <topicName>back_rp/rp_scan_filtered_back/</topicName>
+        <frameName>rp_laser_back</frameName>
+      </plugin>
+    </sensor>
+  </gazebo>
 </robot>

Commit message: Tekerlekler ile zemin arası temas yok

File: wheelchair_description/urdf/wheel_chair.gazebo.xacro (robot description, xacro)
@@ -3,4 +3,5 @@
   <xacro:arg name="laser_visual" default="false"/>
   <xacro:arg name="imu_visual"   default="false"/>
+  <xacro:arg name="camera_name"   default="camera"/>
   <gazebo reference="base_link">
     <material>Gazebo/DarkGrey</material>
@@ -71,5 +72,5 @@
       <wheelDiameter>0.324</wheelDiameter>
       <wheelAcceleration>1</wheelAcceleration>
-      <wheelTorque>50</wheelTorque>
+      <wheelTorque>10</wheelTorque>
       <rosDebugLevel>na</rosDebugLevel>
     </plugin>
@@ -112,14 +113,14 @@
         <scan>
           <horizontal>
-            <samples>360</samples>
+            <samples>400</samples>
             <resolution>1</resolution>
-            <min_angle>0.0</min_angle>
-            <max_angle>6.28319</max_angle>
+            <min_angle>-1.48352</min_angle>
+            <max_angle>1.48352</max_angle>
           </horizontal>
         </scan>
         <range>
-          <min>0.12</min>
-          <max>7.0</max>
-          <resolution>0.015</resolution>
+          <min>0.20</min>
+          <max>8.0</max>
+          <resolution>1</resolution>
         </range>
         <noise>
@@ -144,8 +145,8 @@
         <scan>
           <horizontal>
-            <samples>360</samples>
+            <samples>600</samples>
             <resolution>1</resolution>
-            <min_angle>0.0</min_angle>
-            <max_angle>6.28319</max_angle>
+            <min_angle>0</min_angle>
+            <max_angle>4.71238</max_angle>
           </horizontal>
         </scan>
@@ -153,5 +154,5 @@
           <min>0.12</min>
           <max>7.0</max>
-          <resolution>0.015</resolution>
+          <resolution>1</resolution>
         </range>
         <noise>
@@ -167,3 +168,44 @@
     </sensor>
   </gazebo>
+  <gazebo reference="camera_link">
+    <sensor name="rgbd_camera" type="depth">
+      <update_rate>30</update_rate>
+      <camera>
+        <horizontal_fov>1.047198</horizontal_fov>
+        <image>
+          <width>848</width>
+          <height>480</height>
+          <format>R8G8B8</format>
+        </image>
+        <clip>
+          <near>0.05</near>
+          <far>3</far>
+        </clip>
+      </camera>
+      <plugin name="rgbd_camera_controller" filename="libgazebo_ros_openni_kinect.so">
+        <baseline>0.2</baseline>
+        <alwaysOn>true</alwaysOn>
+        <updateRate>1.0</updateRate>
+        <cameraName>camera_ir</cameraName>
+        <imageTopicName>/camera/color/image_raw</imageTopicName>
+        <cameraInfoTopicName>/camera/color/camera_info</cameraInfoTopicName>
+        <depthImageTopicName>/camera/depth/image_raw</depthImageTopicName>
+        <depthImageInfoTopicName>/camera/depth/camera_info</depthImageInfoTopicName>
+        <pointCloudTopicName>/camera/depth/points</pointCloudTopicName>
+        <frameName>camera_link</frameName>
+        <pointCloudCutoff>0.5</pointCloudCutoff>
+        <pointCloudCutoffMax>3.0</pointCloudCutoffMax>
+        <distortionK1>0.00000001</distortionK1>
+        <distortionK2>0.00000001</distortionK2>
+        <distortionK3>0.00000001</distortionK3>
+        <distortionT1>0.00000001</distortionT1>
+        <distortionT2>0.00000001</distortionT2>
+        <CxPrime>0</CxPrime>
+        <Cx>0</Cx>
+        <Cy>0</Cy>
+        <focalLength>0</focalLength>
+        <hackBaseline>0</hackBaseline>
+      </plugin>
+    </sensor>
+  </gazebo>
 </robot>

File: wheelchair_description/urdf/wheel_chair.urdf.xacro (robot description, xacro)
@@ -3,4 +3,10 @@
   <!-- <xacro:include filename="$(find turtlebot3_description)/urdf/common_properties.xacro" /> -->
   <xacro:include filename="$(find wheelchair_description)/urdf/wheel_chair.gazebo.xacro" />
+  <link name="base_footprint" />
+  <joint name="base_joint" type="fixed">
+    <parent link="base_footprint" />
+    <child link="base_link" />
+    <origin xyz="0.0 0.0 0.0010" rpy="0 0 0" />
+  </joint>
   <link
     name="base_link">
@@ -44,9 +50,9 @@
   </link>
   <joint name="imu_joint" type="fixed">
-    <parent link="base_link"/>
-    <child link="imu_link"/>
-    <origin xyz="-0.032 0 0.068" rpy="0 0 0"/>
-  </joint>
-  <link name="imu_link"/>
+    <parent link="base_link" />
+    <child link="imu_link" />
+    <origin xyz="-0.032 0 0.068" rpy="0 0 0" />
+  </joint>
+  <link name="imu_link" />
   <link
     name="left_big_wheel">
@@ -82,35 +88,25 @@
       <origin
         xyz="0 0 0"
-        rpy="0 0 0" />
-      <geometry>
-        <mesh
-          filename="package://wheel_chair/meshes/left_big_wheel.STL" />
-      </geometry>
-    </collision>
-  </link>
-  <joint
-    name="left_big_wheel_joint"
-    type="continuous">
-    <origin
-      xyz="0 0.315 0"
-      rpy="0 0 0" />
-    <parent
-      link="base_link" />
-    <child
-      link="left_big_wheel" />
-    <axis
-      xyz="0 -1 0" />
-    <limit
-      effort="1"
-      velocity="1" />
-  </joint>
-  <link
-    name="right_big_wheel">
+        rpy="-1.57 0 0" />
+      <geometry>
+        <!-- <mesh
+          filename="package://wheel_chair/meshes/left_big_wheel.STL" /> -->
+          <cylinder length="0.055" radius="0.15"/>
+      </geometry>
+    </collision>
+  </link>
+  <joint name="left_big_wheel_joint" type="continuous">
+    <origin xyz="0 0.315 0" rpy="0 0 0" />
+    <parent link="base_link" />
+    <child link="left_big_wheel" />
+    <axis xyz="0 -1 0" />
+    <!-- <limit effort="1" velocity="1" /> -->
+  </joint>
+  <link name="right_big_wheel">
     <inertial>
       <origin
         xyz="1.60982338570648E-15 0.0275 1.11022302462516E-15"
         rpy="0 0 0" />
-      <mass
-        value="3.19005851775018" />
+      <mass value="3.19005851775018" />
       <inertia
         ixx="0.0222055020892377"
@@ -138,8 +134,9 @@
       <origin
         xyz="0 0 0"
-        rpy="0 0 0" />
-      <geometry>
-        <mesh
-          filename="package://wheel_chair/meshes/right_big_wheel.STL" />
+        rpy="-1.57 0 0" />
+      <geometry>
+        <!-- <mesh
+          filename="package://wheel_chair/meshes/right_big_wheel.STL" /> -->
+          <cylinder length="0.055" radius="0.15"/>
       </geometry>
     </collision>
@@ -194,8 +191,9 @@
       <origin
         xyz="0 0 0"
-        rpy="0 0 0" />
-      <geometry>
-        <mesh
-          filename="package://wheel_chair/meshes/left_small_wheel.STL" />
+        rpy="1.57 0 0" />
+      <geometry>
+        <!-- <mesh
+          filename="package://wheel_chair/meshes/left_small_wheel.STL" /> -->
+          <cylinder length="0.055" radius="0.09"/>
       </geometry>
     </collision>
@@ -252,8 +250,9 @@
       <origin
         xyz="0 0 0"
-        rpy="0 0 0" />
-      <geometry>
-        <mesh
-          filename="package://wheel_chair/meshes/right_smaal_wheel.STL" />
+        rpy="1.57 0 0" />
+      <geometry>
+        <!-- <mesh
+          filename="package://wheel_chair/meshes/right_smaal_wheel.STL" /> -->
+          <cylinder length="0.055" radius="0.09"/>
       </geometry>
     </collision>
@@ -322,5 +321,5 @@
     <origin
       xyz="-0.048279 0.305 0.26099"
-      rpy="0 0 -0.4" />
+      rpy="0 0 0" />
     <parent
       link="base_link" />
@@ -375,5 +374,5 @@
     <origin
       xyz="0.72155 0.0046595 -0.074152"
-      rpy="0 0 -0.0013615" />
+      rpy="0 0 0.0" />
     <parent
       link="base_link" />

Commit message: ön teker sürtünme sıfırlandı yaw açısı eklendi

File: wheelchair_description/urdf/wheel_chair.gazebo.xacro (robot description, xacro)
@@ -28,6 +28,6 @@
   </gazebo>
   <gazebo reference="left_small_wheel">
-    <mu1>0.1</mu1>
-    <mu2>0.1</mu2>
+    <mu1>0.0</mu1>
+    <mu2>0.0</mu2>
     <kp>1000000.0</kp>
     <kd>100.0</kd>
@@ -37,6 +37,6 @@
   </gazebo>
   <gazebo reference="right_smaal_wheel">
-    <mu1>0.1</mu1>
-    <mu2>0.1</mu2>
+    <mu1>0.0</mu1>
+    <mu2>0.0</mu2>
     <kp>1000000.0</kp>
     <kd>100.0</kd>

File: wheelchair_description/urdf/wheel_chair.urdf.xacro (robot description, xacro)
@@ -44,6 +44,7 @@
         rpy="0 0 0" />
       <geometry>
-        <mesh
-          filename="package://wheel_chair/meshes/base_link.STL" />
+        <!-- <mesh
+          filename="package://wheel_chair/meshes/base_link.STL" /> -->
+          <box size="0.8 0.6 0.0" />
       </geometry>
     </collision>
@@ -88,9 +89,10 @@
       <origin
         xyz="0 0 0"
-        rpy="-1.57 0 0" />
+        rpy="-1.5707963268 0 3.1415" />
       <geometry>
         <!-- <mesh
           filename="package://wheel_chair/meshes/left_big_wheel.STL" /> -->
-          <cylinder length="0.055" radius="0.15"/>
+          <cylinder length="0.06" radius="0.16"/>
+          <!-- <cylinder length="0.25" radius="0.25"/> -->
       </geometry>
     </collision>
@@ -134,9 +136,10 @@
       <origin
         xyz="0 0 0"
-        rpy="-1.57 0 0" />
+        rpy="-1.5707963268 0 3.1415" />
       <geometry>
         <!-- <mesh
           filename="package://wheel_chair/meshes/right_big_wheel.STL" /> -->
-          <cylinder length="0.055" radius="0.15"/>
+          <cylinder length="0.06" radius="0.16"/>
+          <!-- <cylinder length="0.25" radius="0.25"/> -->
       </geometry>
     </collision>
@@ -195,5 +198,6 @@
         <!-- <mesh
           filename="package://wheel_chair/meshes/left_small_wheel.STL" /> -->
-          <cylinder length="0.055" radius="0.09"/>
+          <cylinder length="0.055" radius="0.095"/>
+          <!-- <cylinder length="0.25" radius="0.25"/> -->
       </geometry>
     </collision>
@@ -212,8 +216,8 @@
       xyz="-0.0019131 1 0" />
     <limit
-      lower="0"
-      upper="0"
-      effort="0"
-      velocity="0" />
+      lower="0.1"
+      upper="1.0"
+      effort="1"
+      velocity="1" />
   </joint>
   <link
@@ -254,5 +258,6 @@
         <!-- <mesh
           filename="package://wheel_chair/meshes/right_smaal_wheel.STL" /> -->
-          <cylinder length="0.055" radius="0.09"/>
+          <cylinder length="0.055" radius="0.095"/>
+          <!-- <cylinder length="0.25" radius="0.25"/> -->
       </geometry>
     </collision>
@@ -271,8 +276,8 @@
       xyz="0.0043627 0.99999 0" />
     <limit
-      lower="0"
-      upper="0"
-      effort="0"
-      velocity="0" />
+      lower="0.1"
+      upper="1.0"
+      effort="1"
+      velocity="1" />
   </joint>
   <link

Commit message: ileri gidiyor, mu'lar fena degil

File: wheelchair_description/urdf/wheel_chair.gazebo.xacro (robot description, xacro)
@@ -8,39 +8,41 @@
   </gazebo>
   <gazebo reference="left_big_wheel">
+    <mu1>0.4</mu1>
+    <mu2>0.4</mu2>
+    <kp>1000000.0</kp>
+    <kd>100.0</kd>
+    <minDepth>0.001</minDepth>
+    <maxVel>0.5</maxVel>
+    <fdir1>1 0 0</fdir1>
+    <material>Gazebo/FlatBlack</material>
+  </gazebo>
+  <gazebo reference="right_big_wheel">
+    <mu1>0.4</mu1>
+    <mu2>0.4</mu2>
+    <kp>1000000.0</kp>
+    <kd>100.0</kd>
+    <minDepth>0.001</minDepth>
+    <maxVel>0.5</maxVel>
+    <fdir1>1 0 0</fdir1>
+    <material>Gazebo/FlatBlack</material>
+  </gazebo>
+  <gazebo reference="left_small_wheel">
     <mu1>0.1</mu1>
     <mu2>0.1</mu2>
-    <kp>500000.0</kp>
-    <kd>10.0</kd>
-    <minDepth>0.001</minDepth>
-    <maxVel>0.5</maxVel>
-    <fdir1>1 0 0</fdir1>
-    <material>Gazebo/FlatBlack</material>
-  </gazebo>
-  <gazebo reference="right_big_wheel">
+    <kp>1000000.0</kp>
+    <kd>100.0</kd>
+    <minDepth>0.001</minDepth>
+    <maxVel>0.5</maxVel>
+    <fdir1>1 0 0</fdir1>
+    <material>Gazebo/FlatBlack</material>
+  </gazebo>
+  <gazebo reference="right_smaal_wheel">
     <mu1>0.1</mu1>
     <mu2>0.1</mu2>
-    <kp>500000.0</kp>
-    <kd>10.0</kd>
-    <minDepth>0.001</minDepth>
-    <maxVel>0.5</maxVel>
-    <fdir1>1 0 0</fdir1>
-    <material>Gazebo/FlatBlack</material>
-  </gazebo>
-  <gazebo reference="left_small_wheel">
-    <mu1>0.0</mu1>
-    <mu2>0.0</mu2>
-    <kp>1000000.0</kp>
-    <kd>100.0</kd>
-    <minDepth>0.001</minDepth>
-    <maxVel>0.5</maxVel>
-    <material>Gazebo/FlatBlack</material>
-  </gazebo>
-  <gazebo reference="right_smaal_wheel">
-    <mu1>0.0</mu1>
-    <mu2>0.0</mu2>
-    <kp>1000000.0</kp>
-    <kd>100.0</kd>
-    <minDepth>0.001</minDepth>
-    <maxVel>0.5</maxVel>
+    <kp>1000000.0</kp>
+    <kd>100.0</kd>
+    <minDepth>0.001</minDepth>
+    <maxVel>0.5</maxVel>
+    <fdir1>1 0 0</fdir1>
     <material>Gazebo/FlatBlack</material>
   </gazebo>

File: wheelchair_description/urdf/wheel_chair.urdf.xacro (robot description, xacro)
@@ -44,7 +44,7 @@
         rpy="0 0 0" />
       <geometry>
-        <!-- <mesh
-          filename="package://wheel_chair/meshes/base_link.STL" /> -->
-          <box size="0.8 0.6 0.0" />
+        <mesh
+          filename="package://wheel_chair/meshes/base_link.STL" />
+          <!-- <box size="0.8 0.6 0.0" /> -->
       </geometry>
     </collision>
@@ -102,5 +102,5 @@
     <parent link="base_link" />
     <child link="left_big_wheel" />
-    <axis xyz="0 -1 0" />
+    <axis xyz="0 1 0" />
     <!-- <limit effort="1" velocity="1" /> -->
   </joint>
@@ -156,5 +156,5 @@
       link="right_big_wheel" />
     <axis
-      xyz="0 -1 0" />
+      xyz="0 1 0" />
     <limit
       effort="1"

Commit message: tekerler tam donmuyor

File: wheelchair_description/urdf/wheel_chair.gazebo.xacro (robot description, xacro)
@@ -11,7 +11,7 @@
     <mu2>0.4</mu2>
     <kp>1000000.0</kp>
-    <kd>100.0</kd>
-    <minDepth>0.001</minDepth>
-    <maxVel>0.5</maxVel>
+    <kd>100</kd>
+    <minDepth>0.001</minDepth>
+    <maxVel>1</maxVel>
     <fdir1>1 0 0</fdir1>
     <material>Gazebo/FlatBlack</material>
@@ -23,5 +23,5 @@
     <kd>100.0</kd>
     <minDepth>0.001</minDepth>
-    <maxVel>0.5</maxVel>
+    <maxVel>1</maxVel>
     <fdir1>1 0 0</fdir1>
     <material>Gazebo/FlatBlack</material>
@@ -33,5 +33,5 @@
     <kd>100.0</kd>
     <minDepth>0.001</minDepth>
-    <maxVel>0.5</maxVel>
+    <maxVel>1</maxVel>
     <fdir1>1 0 0</fdir1>
     <material>Gazebo/FlatBlack</material>
@@ -43,5 +43,5 @@
     <kd>100.0</kd>
     <minDepth>0.001</minDepth>
-    <maxVel>0.5</maxVel>
+    <maxVel>1</maxVel>
     <fdir1>1 0 0</fdir1>
     <material>Gazebo/FlatBlack</material>

File: wheelchair_description/urdf/wheel_chair.urdf.xacro (robot description, xacro)
@@ -89,9 +89,9 @@
       <origin
         xyz="0 0 0"
-        rpy="-1.5707963268 0 3.1415" />
-      <geometry>
-        <!-- <mesh
-          filename="package://wheel_chair/meshes/left_big_wheel.STL" /> -->
-          <cylinder length="0.06" radius="0.16"/>
+        rpy="0 0 0" />
+      <geometry>
+        <mesh
+          filename="package://wheel_chair/meshes/left_big_wheel.STL" />
+          <!-- <cylinder length="0.06" radius="0.16"/> -->
           <!-- <cylinder length="0.25" radius="0.25"/> -->
       </geometry>
@@ -136,9 +136,9 @@
       <origin
         xyz="0 0 0"
-        rpy="-1.5707963268 0 3.1415" />
-      <geometry>
-        <!-- <mesh
-          filename="package://wheel_chair/meshes/right_big_wheel.STL" /> -->
-          <cylinder length="0.06" radius="0.16"/>
+        rpy="0 0 0" />
+      <geometry>
+        <mesh
+          filename="package://wheel_chair/meshes/right_big_wheel.STL" />
+          <!-- <cylinder length="0.06" radius="0.16"/> -->
           <!-- <cylinder length="0.25" radius="0.25"/> -->
       </geometry>
@@ -194,9 +194,9 @@
       <origin
         xyz="0 0 0"
-        rpy="1.57 0 0" />
-      <geometry>
-        <!-- <mesh
-          filename="package://wheel_chair/meshes/left_small_wheel.STL" /> -->
-          <cylinder length="0.055" radius="0.095"/>
+        rpy="0 0 0" />
+      <geometry>
+        <mesh
+          filename="package://wheel_chair/meshes/left_small_wheel.STL" />
+          <!-- <cylinder length="0.055" radius="0.095"/> -->
           <!-- <cylinder length="0.25" radius="0.25"/> -->
       </geometry>
@@ -217,7 +217,7 @@
     <limit
       lower="0.1"
-      upper="1.0"
-      effort="1"
-      velocity="1" />
+      upper="10.0"
+      effort="10"
+      velocity="100" />
   </joint>
   <link
@@ -254,9 +254,9 @@
       <origin
         xyz="0 0 0"
-        rpy="1.57 0 0" />
-      <geometry>
-        <!-- <mesh
-          filename="package://wheel_chair/meshes/right_smaal_wheel.STL" /> -->
-          <cylinder length="0.055" radius="0.095"/>
+        rpy="0 0 0" />
+      <geometry>
+        <mesh
+          filename="package://wheel_chair/meshes/right_smaal_wheel.STL" />
+          <!-- <cylinder length="0.055" radius="0.095"/> -->
           <!-- <cylinder length="0.25" radius="0.25"/> -->
       </geometry>
@@ -276,8 +276,8 @@
       xyz="0.0043627 0.99999 0" />
     <limit
-      lower="0.1"
+      lower="0.0"
       upper="1.0"
-      effort="1"
-      velocity="1" />
+      effort="0.1"
+      velocity="0.05" />
   </joint>
   <link
