Commit message: Kamera parametreleri güncellendi, frame sorunu çözüldü.

File: wheelchair_description/urdf/wheel_chair.gazebo.xacro (robot description, xacro)
@@ -174,9 +174,16 @@
     </sensor>
   </gazebo>
+  <link name="camera_gazebo" />
+  <joint name="camera_gazebo_joint" type="fixed">
+    <parent link="camera_link"/>
+    <child link="camera_gazebo"/>
+    <origin xyz="0.0 0 0" rpy="-1.5707963267948966 0 -1.5707963267948966"/>
+  </joint>
   <gazebo reference="camera_link">
     <sensor name="rgbd_camera" type="depth">
       <update_rate>30</update_rate>
       <camera>
-        <horizontal_fov>1.047198</horizontal_fov>
+        <horizontal_fov>1.5184351666666667</horizontal_fov>
+        <vertical_fov>1.0122901111111111</vertical_fov>
         <image>
           <width>848</width>
@@ -185,6 +192,6 @@
         </image>
         <clip>
-          <near>0.05</near>
-          <far>3</far>
+          <near>0.01</near>
+          <far>5.0</far>
         </clip>
       </camera>
@@ -192,6 +199,6 @@
         <baseline>0.2</baseline>
         <alwaysOn>true</alwaysOn>
-        <updateRate>1.0</updateRate>
-        <cameraName>camera_ir</cameraName>
+        <updateRate>30.0</updateRate>
+        <cameraName>camera</cameraName>
         <imageTopicName>/camera/color/image_raw</imageTopicName>
         <cameraInfoTopicName>/camera/color/camera_info</cameraInfoTopicName>
@@ -199,7 +206,7 @@
         <depthImageInfoTopicName>/camera/depth/camera_info</depthImageInfoTopicName>
         <pointCloudTopicName>/camera/depth/points</pointCloudTopicName>
-        <frameName>camera_link</frameName>
-        <pointCloudCutoff>0.5</pointCloudCutoff>
-        <pointCloudCutoffMax>3.0</pointCloudCutoffMax>
+        <frameName>camera_gazebo</frameName>
+        <pointCloudCutoff>0.2</pointCloudCutoff>
+        <pointCloudCutoffMax>5.0</pointCloudCutoffMax>
         <distortionK1>0.00000001</distortionK1>
         <distortionK2>0.00000001</distortionK2>

File: wheelchair_description/urdf/wheel_chair.urdf (robot description, URDF)
Before this commit: robot wheel_chair, 21 links, 20 joints
Joints:
- joint camera_color_optical_joint: origin xyz=0 0 0 rpy=-1.57079632679 0 -1.57079632679 -> xyz=0 0 0 rpy=0 0 0
- joint camera_depth_optical_joint: origin xyz=0 0 0 rpy=-1.57079632679 0 -1.57079632679 -> xyz=0 0 0 rpy=0 0 0
- joint camera_infra1_optical_joint: origin xyz=0 0 0 rpy=-1.57079632679 0 -1.57079632679 -> xyz=0 0 0 rpy=0 0 0
- joint camera_infra2_optical_joint: origin xyz=0 0 0 rpy=-1.57079632679 0 -1.57079632679 -> xyz=0 0 0 rpy=0 0 0; parent camera_infra2_frame -> (none)
- joint camera_joint: origin xyz=-0.066986 -0.0039691 1.5345 rpy=0 0 0 -> xyz=-0.066986 -0.0039691 1.5345 rpy=-1.57 -1.57 -1.57

File: wheelchair_description/urdf/wheel_chair.urdf.xacro (robot description, xacro)
@@ -453,4 +453,5 @@
   <joint name="camera_depth_optical_joint" type="fixed">
     <origin xyz="0 0 0" rpy="-1.57079632679 0 -1.57079632679" />
+    <!-- <origin xyz="0 0 0" rpy="0 0 0" /> -->
     <parent link="camera_depth_frame" />
     <child link="camera_depth_optical_frame" />
@@ -466,4 +467,5 @@
   <joint name="camera_infra1_optical_joint" type="fixed">
     <origin xyz="0 0 0" rpy="-1.57079632679 0 -1.57079632679" />
+    <!-- <origin xyz="0 0 0" rpy="0 0 0" /> -->
     <parent link="camera_infra1_frame" />
     <child link="camera_infra1_optical_frame" />
@@ -479,4 +481,5 @@
   <joint name="camera_infra2_optical_joint" type="fixed">
     <origin xyz="0 0 0" rpy="-1.57079632679 0 -1.57079632679" />
+    <!-- <origin xyz="0 0 0" rpy="0 0 0" /> -->
     <parent link="camera_infra2_frame" />
     <child link="camera_infra2_optical_frame" />
@@ -492,4 +495,5 @@
   <joint name="camera_color_optical_joint" type="fixed">
     <origin xyz="0 0 0" rpy="-1.57079632679 0 -1.57079632679" />
+    <!-- <origin xyz="0 0 0" rpy="0 0 0" /> -->
     <parent link="camera_color_frame" />
     <child link="camera_color_optical_frame" />

Commit message: Actor senaryolarına hız seçenekleri eklendi ve iyileştirildi.

File: wheelchair_description/urdf/wheel_chair.gazebo.xacro (robot description, xacro)
@@ -7,5 +7,5 @@
     <material>Gazebo/DarkGrey</material>
   </gazebo>
-  <gazebo reference="left_big_wheel">
+  <!-- <gazebo reference="left_big_wheel">
     <mu1>0.4</mu1>
     <mu2>0.4</mu2>
@@ -14,8 +14,8 @@
     <minDepth>0.0</minDepth>
     <maxVel>0.1</maxVel>
-    <!-- <fdir1>1 0 0</fdir1> -->
-    <material>Gazebo/FlatBlack</material>
-  </gazebo>
-  <gazebo reference="right_big_wheel">
+    <fdir1>1 0 0</fdir1>
+    <material>Gazebo/FlatBlack</material>
+  </gazebo> -->
+  <!-- <gazebo reference="right_big_wheel">
     <mu1>0.4</mu1>
     <mu2>0.4</mu2>
@@ -24,7 +24,7 @@
     <minDepth>0.0</minDepth>
     <maxVel>0.1</maxVel>
-    <!-- <fdir1>1 0 0</fdir1> -->
-    <material>Gazebo/FlatBlack</material>
-  </gazebo>
+    <fdir1>1 0 0</fdir1>
+    <material>Gazebo/FlatBlack</material>
+  </gazebo> -->
   <gazebo reference="left_small_wheel">
     <mu1>0.0</mu1>

Commit message: people_tracker paketine revize geldi.

File: wheelchair_description/urdf/wheel_chair.gazebo.xacro (robot description, xacro)
@@ -7,5 +7,5 @@
     <material>Gazebo/DarkGrey</material>
   </gazebo>
-  <!-- <gazebo reference="left_big_wheel">
+  <gazebo reference="left_big_wheel">
     <mu1>0.4</mu1>
     <mu2>0.4</mu2>
@@ -14,8 +14,8 @@
     <minDepth>0.0</minDepth>
     <maxVel>0.1</maxVel>
-    <fdir1>1 0 0</fdir1>
-    <material>Gazebo/FlatBlack</material>
-  </gazebo> -->
-  <!-- <gazebo reference="right_big_wheel">
+    <!-- <fdir1>1 0 0</fdir1> -->
+    <material>Gazebo/FlatBlack</material>
+  </gazebo>
+  <gazebo reference="right_big_wheel">
     <mu1>0.4</mu1>
     <mu2>0.4</mu2>
@@ -24,7 +24,7 @@
     <minDepth>0.0</minDepth>
     <maxVel>0.1</maxVel>
-    <fdir1>1 0 0</fdir1>
-    <material>Gazebo/FlatBlack</material>
-  </gazebo> -->
+    <!-- <fdir1>1 0 0</fdir1> -->
+    <material>Gazebo/FlatBlack</material>
+  </gazebo>
   <gazebo reference="left_small_wheel">
     <mu1>0.0</mu1>

Commit message: anamiz agladi ama collision verisi aliniyor, loglaniyor, gazebo_ros paketleri yüklendi contact sensorler eklendi urdf xacro ve gazebo xacro buyuk olcude degisti

File: wheelchair_description/urdf/wheel_chair.gazebo.xacro (robot description, xacro)
@@ -4,6 +4,31 @@
   <xacro:arg name="imu_visual"   default="false"/>
   <xacro:arg name="camera_name"   default="camera"/>
+  <gazebo reference="base_footprint">
+    <material>Gazebo/DarkGrey</material>
+    <sensor name="base_footprint_contact_sensor" type="contact">
+      <always_on>true</always_on>
+      <update_rate>10</update_rate>
+      <contact>
+        <collision>base_footprint_collision</collision>
+      </contact>
+      <plugin name="base_footprint_bumper" filename="libgazebo_ros_bumper.so">
+        <bumperTopicName>base_footprint_contact_sensor_state</bumperTopicName>
+        <frameName>base_footprint</frameName>
+      </plugin>
+    </sensor>
+  </gazebo>
   <gazebo reference="base_link">
     <material>Gazebo/DarkGrey</material>
+    <sensor name="base_link_contact_sensor" type="contact">
+      <always_on>true</always_on>
+      <update_rate>10</update_rate>
+      <contact>
+        <collision>base_link_collision</collision>
+      </contact>
+      <plugin name="base_link_bumper" filename="libgazebo_ros_bumper.so">
+        <bumperTopicName>base_link_contact_sensor_state</bumperTopicName>
+        <frameName>base_link</frameName>
+      </plugin>
+    </sensor>
   </gazebo>
   <gazebo reference="left_big_wheel">
@@ -16,4 +41,15 @@
     <!-- <fdir1>1 0 0</fdir1> -->
     <material>Gazebo/FlatBlack</material>
+    <sensor name="left_big_wheel_contact_sensor" type="contact">
+      <always_on>true</always_on>
+      <update_rate>10</update_rate>
+      <contact>
+        <collision>left_big_wheel_collision</collision>
+      </contact>
+      <plugin name="left_big_wheel_bumper" filename="libgazebo_ros_bumper.so">
+        <bumperTopicName>left_big_wheel_contact_sensor_state</bumperTopicName>
+        <frameName>left_big_wheel</frameName>
+      </plugin>
+    </sensor>
   </gazebo>
   <gazebo reference="right_big_wheel">
@@ -26,4 +62,15 @@
     <!-- <fdir1>1 0 0</fdir1> -->
     <material>Gazebo/FlatBlack</material>
+    <sensor name="right_big_wheel_contact_sensor" type="contact">
+      <always_on>true</always_on>
+      <update_rate>10</update_rate>
+      <contact>
+        <collision>right_big_wheel_collision</collision>
+      </contact>
+      <plugin name="right_big_wheel_bumper" filename="libgazebo_ros_bumper.so">
+        <bumperTopicName>right_big_wheel_contact_sensor_state</bumperTopicName>
+        <frameName>right_big_wheel</frameName>
+      </plugin>
+    </sensor>
   </gazebo>
   <gazebo reference="left_small_wheel">
@@ -36,4 +83,15 @@
     <!-- <fdir1>1 0 0</fdir1> -->
     <material>Gazebo/FlatBlack</material>
+    <sensor name="left_small_wheel_contact_sensor" type="contact">
+      <always_on>true</always_on>
+      <update_rate>10</update_rate>
+      <contact>
+        <collision>left_small_wheel_collision</collision>
+      </contact>
+      <plugin name="left_small_wheel_bumper" filename="libgazebo_ros_bumper.so">
+        <bumperTopicName>left_small_wheel_contact_sensor_state</bumperTopicName>
+        <frameName>left_small_wheel</frameName>
+      </plugin>
+    </sensor>
   </gazebo>
   <gazebo reference="right_smaal_wheel">
@@ -46,4 +104,15 @@
     <!-- <fdir1>1 0 0</fdir1> -->
     <material>Gazebo/FlatBlack</material>
+    <sensor name="right_smaal_wheel_contact_sensor" type="contact">
+      <always_on>true</always_on>
+      <update_rate>10</update_rate>
+      <contact>
+        <collision>right_smaal_wheel_collision</collision>
+      </contact>
+      <plugin name="right_smaal_wheel_bumper" filename="libgazebo_ros_bumper.so">
+        <bumperTopicName>right_smaal_wheel_contact_sensor_state</bumperTopicName>
+        <frameName>right_smaal_wheel</frameName>
+      </plugin>
+    </sensor>
   </gazebo>
   <gazebo reference="imu_link">

File: wheelchair_description/urdf/wheel_chair.urdf.xacro (robot description, xacro)
@@ -4,14 +4,51 @@
   <xacro:include filename="$(find wheelchair_description)/urdf/wheel_chair.gazebo.xacro" />
   <link name="base_footprint" >
-    <visual>
+    <inertial>
+      <origin
+        xyz="8.32667268468867E-17 -0.0275 9.43689570931383E-16"
+        rpy="0 0 0" />
+      <mass
+        value="0.1" />
+      <inertia
+        ixx="0.0222055020892376"
+        ixy="2.73068863816006E-19"
+        ixz="-2.79570503430672E-17"
+        iyy="0.0429444812918596"
+        iyz="-3.90098376880016E-20"
+        izz="0.0222055020892377" />
+    </inertial>
+    <visual>
+      <origin
+        xyz="0 0 0"
+        rpy="0 0 0" />
       <geometry>
         <cylinder length = "0.2" radius="0.05" />
       </geometry>
-    </visual>
+      <material
+        name="">
+        <color
+          rgba="0.298039215686275 0.298039215686275 0.298039215686275 1" />
+      </material>
+    </visual>
+    <collision>
+      <origin
+        xyz="-0.4 0 0.15345"
+        rpy="0 0 0" /> <!-- contact sensorle ilgili ypailmis degisikliklerden oturu sorun cikarsa burda cok sey degisecek direkt 11 temmuz 2023 lü github versiyonuna döndür -->
+      <geometry>
+        <mesh
+          filename="package://wheel_chair/meshes/base_link.STL" />
+      </geometry>
+    </collision>
+    <!-- <visual>
+      <geometry>
+        <cylinder length = "0.2" radius="0.05" /> Contact icin yapilmis footprint degisikligi geri alindiginda bu commentli kisim aktif edilecek
+      </geometry>
+    </visual> -->
 </link>
   <joint name="base_joint" type="fixed">
     <parent link="base_footprint" />
     <child link="base_link" />
-    <origin xyz="-0.40 0.0 0.15345" rpy="0 0 0" />
+    <!-- <origin xyz="-0.40 0.0 -0.14655" rpy="0 0 0" /> -->
+    <origin xyz="-0.40 0.0 0.15345" rpy="0 0 0" /><!--Bu contact icin yapilmis footprint degisikligi geri alindiginda aktif edilecek -->
   </joint>
   <link
@@ -52,5 +89,5 @@
         <mesh
           filename="package://wheel_chair/meshes/base_link.STL" />
-          <!-- <box size="0.8 0.6 0.0" /> -->
+          <!-- <box size="0.8 0.6 1.0" /> -->
       </geometry>
     </collision>
